File: H2BR0-5/Design/H2BR0-5.sch (EAGLE design)
At the start: 62 parts, among them J1 CUI_DEVICES_SJ-3524-SMT-TRCUI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, P2 HEXABIT_X2_P1_P5, U1 STM32G0B1CEU6QFN_B1CEU6_STM-L, U2 AD8232ACPZ-WP, U3 MCP6002, X1 XTALL_CSTCE8M00G52

Commit message: -The final design, all done.
Parts:
- removed C14: 1uF, HEXABITZ_RCLS:C-0805-POL
- added C5: 1uF, HEXABITZ_RCLS:C-0402
- added J3: 440054-3, HEXABITZ_CONNECTION_PARTS:440054-3
- added R28: 100k, HEXABITZ_RCLS:R-0402
- added R29, R30: (no value), HEXABITZ_RCLS:SB-0603
- added R31: 22K, HEXABITZ_RCLS:R-0402
- added SH1: SMS-202C, HEXABITZ_OTHER_PARTS:SMS-202C
- C10, C11, C12, C13, C15, C16, C17, C18, C19, C21, C8, C9: device HEXABITZ_RCLS:C-0603 -> HEXABITZ_RCLS:C-0402
- C20: value 1uF -> 100nF; device HEXABITZ_RCLS:C-0603 -> HEXABITZ_RCLS:C-0402
- J1: value CUI_DEVICES_SJ-3524-SMT-TRCUI_DEVICES_SJ-3524-SMT-TR_0_0 -> SJ-3524-SMT-TRU; device HEXABITZ_ICs:CUI_DEVICES_SJ-3524-SMT-TRCUI_DEVICES_SJ-3524-SMT-TR_0_0 -> HEXABITZ_ICs:SJ-3524-SMT-TRU
- R10, R11, R12, R13, R14, R15, R16, R17, R18, R19, R20, R21, R22, R23, R24, R25, R4, R5, R6, R7, R8, R9: device HEXABITZ_RCLS:R-0603 -> HEXABITZ_RCLS:R-0402
- R27: value 0R -> 200k; device HEXABITZ_RCLS:R-0603 -> HEXABITZ_RCLS:R-0402
- U2: value AD8232ACPZ-WP -> AD8232ACPZ-R7; device HEXABITZ_ICs:AD8232ACPZ-WP -> HEXABITZ_ICs:AD8232ACPZ-R7
- U3: value MCP6002 -> TSV772IQ2T_SEPARATED_SYMBOLSSON50P200X200X60-9N; device HEXABITZ_ICs:MCP6002-I/SNSOIC8-N_MC_MCH-L -> HEXABITZ_ICs:TSV772IQ2T_SEPARATED_SYMBOLSSON50P200X200X60-9N
Connections:
- removed net N$28: C18.2, C19.2, R20.1, R21.2
- removed net N$3 (its old number): C21.1, R4.1, R5.2, U2.REFIN
- removed net REFOUT: C10.1, C13.2, R16.2, R24.2, R25.1, U2.REFOUT
- removed net SW: C10.2, R8.2, U2.SW
- removed net USART6_RX: P2.SD1, U1.PB9
- removed net USART6_TX: P2.SU1, U1.PB8
- new net N$11: R18.2, S1.6, S1.7
- new net N$12: C12.2, R14.1, R15.1, S1.1, S1.5
- new net N$14: C9.1, R6.2, U2.HPSENSE
- new net N$21: C17.1, R20.2, U3(1).+IN
- new net N$29: C11.2, U2.RLDFB
- new net USART4_RX: P2.SD3, U1.PA1
- new net USART4_TX: P2.SU3, U1.PA0
- net GND: no longer C14.-, C15.2, C21.2, C8.2, D2.C, JP4.2, R22.1, R5.1, U2.AC/!DC, U2.GND, U2.GND_EP, U3.VSS
- net IN+: now also J1.3, J3.3; no longer J1.RING
- net IN-: now also J1.1, J3.2; no longer J1.SLEEVE
- net LOD+: now also U1.PB8; no longer U1.PA7
- net LOD-: now also U1.PB7; no longer U1.PB0
- net N$10: now also R19.1, S1.2, S1.3; no longer R6.2, R7.2, R8.1
- net N$13: now also R15.2, R18.1, R7.1, U2.IAOUT; no longer C11.1, U2.RLDFB
- net N$16: now also R6.1, R7.2, R8.1; no longer C12.2, R14.2, R15.1, S1.3, S1.7
- net N$17: now also R23.2, R24.2, U3(1).-IN; no longer C11.2, R13.1, U2.RLD
- net N$18: now also C21.1, R4.1, R5.1, U2.REFIN; no longer C13.1, R14.1, R19.1, U2.OPAMP+
- net N$19: now also C18.1, C19.1, R20.1, R21.2; no longer R18.1, S1.5, S1.6
- net N$2: now also U1.PA8; no longer U1.PB7
- net N$20: now also C11.1, R13.1, U2.RLD; no longer R19.2, S1.1, S1.2
- net N$22: now also C18.2, C19.2, C20.2, R23.1, R29.2, U3(1).OUT; no longer C17.1, R20.2, U3.VINA+
- net N$23: now also C16.1, C17.2, R22.1; no longer D2.A, R26.1
- net N$24: now also C20.1, R25.2, R29.1, U3(2).+IN; no longer C16.1, C17.2, R22.2
- net N$25: now also C10.2, C13.2, R16.2, R24.1, R25.1, R28.2, U2.REFOUT; no longer C20.2, R25.2, R27.2, U3.VINB+
- net N$26: now also C10.1, R8.2, U2.SW; no longer C18.1, C19.1, C20.1, R23.1, R27.1, U3.VOUTA
- net N$27: now also D2.A, R26.2; no longer R23.2, R24.1, U3.VINA-
- net N$7: now also C13.1, R14.2, R19.2, U2.OPAMP+; no longer C9.1, R6.1, U2.HPSENSE
- net N$9: now also R27.1, R28.1, R30.2, U3(2).-IN; no longer R15.2, R18.2, R7.1, U2.IAOUT
- net OUT: now also R26.1, R27.2, R30.1, U1.PB12, U3(2).OUT; no longer R26.2, U1.PA4, U3.VINB-, U3.VOUTB
- net REF: now also J1.2, J3.1; no longer J1.TIP
- net SDN: now also R31.2, U1.PB9; no longer U1.PA6
- net USART1_RX: now also P2.SD2; no longer P2.SD4
- net USART1_TX: now also P2.SU2; no longer P2.SU4
- net USART2_RX: now also P2.SD4; no longer P2.SD2
- net USART2_TX: now also P2.SU4; no longer P2.SU2
- net USART3_RX: now also P2.SD1; no longer P2.SD3
- net USART3_TX: now also P2.SU1; no longer P2.SU3
- net USART5_RX: now also U1.PB1; no longer U1.PD2
- net USART5_TX: now also U1.PB0; no longer U1.PD3
- net VDD: now also R31.1
- net VDDA: now also C5.1, U3P.V+; no longer C14.+, U3.VDD
- net VSSA: now also C15.2, C21.2, C5.2, C8.2, D2.C, JP4.2, R22.2, R5.2, SH1.SHIELD, U2.AC/!DC, U2.GND, U3P.V-
Other:
- note added: "Desolder R29 for EEG(Alpha)"
- note added: "Desolder R30 for EEG"
- note added: "EXG Monitor (EU Version)"
- note added: "Front End Total Gain =780 HPF: Cut-off freq = 0.048Hz LPF: Cut-off freq = 40Hz for ECG-EOG-EEG Cut-off freq = 160Hz for EMG"
- note added: "H2BR0-5"
- note added: "HPF filter Cut-off freq = 5Hz"
- note added: "Non-Inverting Amplifier Gain=3"
- note added: "Notch filter 50Hz Gain = 1.47"
- note removed: "DNP"
- note removed: "EXG Monitor"
- note removed: "H2BR0"
- moved on the sheet: C1, C10, C11, C12, C13, C15, C16, C17, C18, C19, C2, C20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
