File: H2BR0-6/Design/H2BR0-6.brd (EAGLE design)
At the start: 60 x 34.6 mm, 68 parts, among them J1 SJ-3524-SMT-TRU, J3 440054-3, P2 HEXABIT_X2_P1_P5, U1 STM32G0B1CEU6QFN_B1CEU6_STM-L, U2 AD8232ACPZ-R7, U3 TSV772IQ2T_SEPARATED_SYMBOLSS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, X1 XTALL_CSTCE8M00G52

Commit message: Adding the 60Hz version.
Parts:
- R20, R21: value 32K -> 26.4K
- R22: value 16K -> 13.2K
Other:
- board text added: "H2BR01-6"
- board text removed: "H2BR01-5"
Changed lines of the file:
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@@
 <drawing>
 <settings>
-<setting alwaysvectorfont="yes"/>
+<setting alwaysvectorfont="no"/>
 <setting verticaltext="up"/>
 </settings>
@@
 <text x="-6.588125" y="-11.1125" size="1.9304" layer="26" rot="MR0">P3</text>
 <text x="-9.2075" y="-11.1125" size="1.9304" layer="21">P3</text>
-<text x="23.76678125" y="-0.102615625" size="1.9304" layer="22" font="vector" rot="MR270" align="center">H2BR01-5</text>
+<text x="23.76678125" y="-0.102615625" size="1.9304" layer="22" font="vector" rot="MR270" align="center">H2BR01-6</text>
 <text x="-18.415" y="-3.4925" size="1.9304" layer="21">R</text>
 <text x="-18.415" y="1.666875" size="1.9304" layer="21">C</text>
@@
 <attribute name="VOLTAGE_RATING" value="" x="12.461875" y="2.8575" size="1.778" layer="28" rot="MR0" display="off"/>
 </element>
-<element name="R20" library="HEXABITZ_RCLS" library_urn="urn:adsk.eagle:library:20064561" package="R-0402" package3d_urn="urn:adsk.eagle:package:19666455/4" value="32K" x="6.905625" y="3.01625" smashed="yes" rot="MR90">
+<element name="R20" library="HEXABITZ_RCLS" library_urn="urn:adsk.eagle:library:20064561" package="R-0402" package3d_urn="urn:adsk.eagle:package:19666455/4" value="26.4K" x="6.905625" y="3.01625" smashed="yes" rot="MR90">
 <attribute name="MFN" value="" x="6.905625" y="3.01625" size="1.778" layer="28" rot="MR90" display="off"/>
 <attribute name="MPN" value="" x="6.905625" y="3.01625" size="1.778" layer="28" rot="MR90" display="off"/>
@@
 <attribute name="TOLERANCE" value="" x="6.905625" y="3.01625" size="1.778" layer="28" rot="MR90" display="off"/>
 </element>
-<element name="R21" library="HEXABITZ_RCLS" library_urn="urn:adsk.eagle:library:20064561" package="R-0402" package3d_urn="urn:adsk.eagle:package:19666455/4" value="32K" x="6.19125" y="1.27" smashed="yes" rot="MR180">
+<element name="R21" library="HEXABITZ_RCLS" library_urn="urn:adsk.eagle:library:20064561" package="R-0402" package3d_urn="urn:adsk.eagle:package:19666455/4" value="26.4K" x="6.19125" y="1.27" smashed="yes" rot="MR180">
 <attribute name="MFN" value="" x="6.19125" y="1.27" size="1.778" layer="28" rot="MR180" display="off"/>
 <attribute name="MPN" value="" x="6.19125" y="1.27" size="1.778" layer="28" rot="MR180" display="off"/>
@@
 <attribute name="VOLTAGE_RATING" value="" x="10.00125" y="2.619375" size="1.778" layer="28" rot="MR90" display="off"/>
 </element>
-<element name="R22" library="HEXABITZ_RCLS" library_urn="urn:adsk.eagle:library:20064561" package="R-0402" package3d_urn="urn:adsk.eagle:package:19666455/4" value="16K" x="4.1275" y="4.1275" smashed="yes" rot="MR0">
+<element name="R22" library="HEXABITZ_RCLS" library_urn="urn:adsk.eagle:library:20064561" package="R-0402" package3d_urn="urn:adsk.eagle:package:19666455/4" value="13.2K" x="4.1275" y="4.1275" smashed="yes" rot="MR0">
 <attribute name="MFN" value="" x="4.1275" y="4.1275" size="1.778" layer="28" rot="MR0" display="off"/>
 <attribute name="MPN" value="" x="4.1275" y="4.1275" size="1.778" layer="28" rot="MR0" display="off"/>
